File: hardware/BME680-Breakout_v10.brd (EAGLE design)
At the start: 20 x 20 mm, 23 parts, among them IC1 BME680, IC2 LDO-TS9011-3V3, J1 JUMPER2-0603, T1 BSS138PS, T2 BSS138PS, X1 PASSER-07, X2 PASSER-07

Commit message: updated layout and schematic
Parts:
- renumbered HOUSING1 to HOUSING
Changed lines of the file:
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@@
 <attribute name="NAME" x="6.2865" y="4.445" size="0.8128" layer="21" font="vector" ratio="15" align="center"/>
 </element>
-<element name="HOUSING1" library="we-sensor" package="SF2" value="SF2" x="4.7625" y="9.8425"/>
+<element name="HOUSING" library="we-sensor" package="SF2" value="SF2" x="4.7625" y="9.8425"/>
 <element name="IC1" library="we-sensor" package="BME680" value="BME680" x="4.7625" y="9.8425"/>
 </elements>
